File: KiCad/schematic.kicad_pcb (KiCad board)
At the start: 2 copper layers, 1.4 x 13 mm, 9 parts

Commit message: update CAD
Parts:
- removed the REF** at (33.9, 40.6)
- removed the REF** at (152.5, 70.5)
- removed the REF** at (20.3, 71.1)
- removed the REF** at (88.9, 81.3)
- added J2: Barrel_Jack_Switch, Connector_BarrelJack:BarrelJack_GCT_DCJ200-10-A_Horizontal, F.Cu at (29.8, 87.8)
- added Mic1: INMP441, footprints:INMP441, F.Cu at (46.1, 90.6)
- added U1: ~, ESP32_15x2_header:CJMCU_FT232H, F.Cu at (64.4, 140.4)
- added U2: ~, ESP32_15x2_header:ESP32-DOIT-DEVKIT, F.Cu at (87.4, 91.6)
- moved REF** 72.2 mm to (84.6, 79.1)
- moved REF** 60.2 mm to (69.5, 79.4)
- moved REF** 34.5 mm to (19.8, 97.7)
- moved REF** 28.9 mm to (20.0, 115.1)
- moved REF** 24.5 mm to (20.1, 131.1)
Connections:
- REF** pad 1: (no net) -> +5V
- REF** pad 2: (no net) -> GND
- REF** pad 1: (no net) -> GND
- REF** pad 3: (no net) -> VDD
- REF** pad MP: (no net) -> GND
Routing:
- net (no net): track 1952.1 -> 487.2 mm, vias 13 -> 2
- net +5V: track 0.00 -> 132.1 mm
- net VDD: track 0.00 -> 117.0 mm, vias 0 -> 1
- net GND: track 0.00 -> 105.1 mm, vias 0 -> 1
- net Net-(Mic1-WS): track 0.00 -> 90.0 mm
- added copper zone on B.Cu, net GND
- added copper zone on F.Cu, net GND
